File: pcb/feather-stm32g0b1.kicad_pcb (KiCad board)
At the start: 4 copper layers, 50.8 x 22.9 mm, 50 parts, among them CN1 STDC14, CN2 SM04B-SRSS-TB (LF)(SN), CN3 ZX-PH2.0-WT2P, CN4 SM04B-SRSS-TB (LF)(SN), J1 Conn_01x12, J2 Conn_01x16, J3 GT-USB-7010ASV, Q1 DMG3415U-7, SW1 SW_Push, U1 STM32G0B1CBT6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

Commit message: Added I2C pull ups, extra bypass capacitance for the MCU and increased the LDO output capacitance
Parts:
- added C9: 100nF, Capacitor_SMD:C_0402_1005Metric, B.Cu at (127.5, 91.0)
- added R12: 5K1, Resistor_SMD:R_0402_1005Metric, B.Cu at (148.8, 94.5)
- added R13: 5K1, Resistor_SMD:R_0402_1005Metric, B.Cu at (148.8, 92.2)
- added R14: 5K1, Resistor_SMD:R_0402_1005Metric, B.Cu at (148.8, 88.0)
- added R15: 5K1, Resistor_SMD:R_0402_1005Metric, B.Cu at (148.8, 85.2)
- C2: value 1uF -> 10uF
Connections:
- C7 pad 1: +3V3 -> GND
- C7 pad 2: GND -> +3V3
Routing:
- net +3V3: track 98.0 -> 112.9 mm, vias 8 -> 9
- net I2C2_SCL: track 20.2 -> 23.8 mm, vias 2 -> 3
- net I2C2_SDA: track 19.8 -> 23.3 mm, vias 2 -> 3
- net I2C1_SDA: track 19.6 -> 22.9 mm, vias 2 -> 3
- net I2C1_SCL: track 17.6 -> 20.9 mm, vias 2 -> 3
- net GND: track 47.6 -> 47.9 mm, vias 30 -> 29

Commit message: More PCB layout updates
Parts:
- D4: moved to B.Cu
- moved D4 14.4 mm to (103.2, 91.0), turned to 0 degrees
- turned C7 to 0 degrees
Connections:
- net Net-(D4-I/O1-Pad1) renamed /Power/USBC_DN
- net Net-(D4-I/O2-Pad3) renamed /Power/USBC_DP
- net USB_DM renamed USB_DN
Routing:
- net /Power/USBC_DN: track 22.7 -> 4.06 mm, vias 3 -> 1
- net USB_DP: track 18.6 -> 37.2 mm
- net USB_DN: track 21.2 -> 35.5 mm
- net /Power/USBC_DP: track 18.3 -> 5.02 mm, vias 2 -> 1
- net VBUS: track 60.9 -> 52.7 mm, vias 4 -> 3
- net UART_TX: track 26.7 -> 32.8 mm
- net ANALOG1: track 19.0 -> 18.3 mm
- net +3V3: track 112.9 -> 112.2 mm, vias 9 -> 8
- net SPI_SCK: track 14.7 -> 15.3 mm
- net GND: track 47.9 -> 48.4 mm, vias 29 -> 33
